File: cuteBot.kicad_pcb (KiCad board)
At the start: 2 copper layers, 39.9 x 39.9 mm, 63 parts, among them P1 USB_A, P2 BAT+, P3 BAT-, P4 MOTOR_A, P5 MOTOR_B, P6 CONN_02X03, Q1 S8050, SW1 SW_SPDT, SW2 SW_Push, SW3 SW_Push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

Commit message: 26 nets restantes
Parts:
- L1, U5: moved to F.Cu
- R7: moved to B.Cu
- moved R7 57.4 mm to (148.4, 143.8)
- moved R1 55.4 mm to (147.3, 137.4), turned to 270 degrees
- moved U2 55.0 mm to (151.8, 136.0), turned to 0 degrees
- moved U5 47.7 mm to (144.8, 144.5), turned to 180 degrees
- moved P3 45.3 mm to (150.7, 142.3)
- moved L1 44.8 mm to (151.1, 144.7), turned to 270 degrees
- moved R4 38.9 mm to (148.0, 140.0), turned to 0 degrees
- moved R6 38.1 mm to (150.2, 144.9), turned to 90 degrees
- moved D1 37.8 mm to (154.6, 143.3), turned to 90 degrees
- moved C2 37.4 mm to (144.3, 141.6), turned to 0 degrees
- moved U3 37.2 mm to (144.3, 138.8), turned to 0 degrees
- moved U4 35.7 mm to (144.8, 144.5), turned to 180 degrees
- moved D2 35.0 mm to (154.6, 140.3), turned to 270 degrees
- moved R2 35.0 mm to (153.1, 143.1), turned to 270 degrees
- moved R3 32.2 mm to (153.1, 140.3), turned to 90 degrees
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Routing:
- net Vusb: track 3.95 -> 46.9 mm, vias 0 -> 3
- net GND: track 38.6 -> 52.6 mm, vias 6 -> 13
- net Net-(C2-Pad2): track 0.00 -> 12.7 mm
- net Net-(P2-Pad1): track 0.00 -> 9.92 mm
- net Net-(U3-Pad3): track 0.00 -> 9.90 mm, vias 0 -> 2
- net Net-(R2-Pad1): track 0.00 -> 9.72 mm
- net Net-(C3-Pad1): track 2.25 -> 11.8 mm
- net Net-(U3-Pad1): track 0.00 -> 9.53 mm, vias 0 -> 2
- net 3.3V: track 2.90 -> 10.5 mm
- net Net-(D3-Pad2): track 0.00 -> 7.32 mm
- net Net-(R3-Pad1): track 0.00 -> 6.76 mm
- net Net-(C2-Pad1): track 0.00 -> 6.64 mm
- net Net-(R6-Pad2): track 0.00 -> 6.33 mm, vias 0 -> 1
- net 5V: track 85.3 -> 88.9 mm
- net Net-(C7-Pad2): track 0.00 -> 3.61 mm
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
Commit message: Enrutado comleto
Parts:
- added REF**: MountingHole_3.2mm_M3, Mounting_Holes:MountingHole_3.2mm_M3, F.Cu at (156.2, 152.4)
- added REF**: MountingHole_3.2mm_M3, Mounting_Holes:MountingHole_3.2mm_M3, F.Cu at (121.4, 152.4)
- added REF**: MountingHole_3.2mm_M3, Mounting_Holes:MountingHole_3.2mm_M3, F.Cu at (121.4, 117.6)
- added REF**: MountingHole_3.2mm_M3, Mounting_Holes:MountingHole_3.2mm_M3, F.Cu at (156.2, 117.6)
- C17, C18, C3, C4, U8: moved to F.Cu
- D3: moved to B.Cu
- moved C3 54.3 mm to (153.7, 137.5), turned to 90 degrees
- moved C18 47.6 mm to (138.5, 144.9), turned to 180 degrees
- moved U8 43.7 mm to (138.5, 147.6)
- moved C17 41.4 mm to (141.5, 147.6), turned to 90 degrees
- moved C4 41.3 mm to (146.2, 139.6), turned to 180 degrees
- moved D3 15.8 mm to (153.4, 148.5), turned to 270 degrees
- moved C15 1.07 mm to (144.2, 124.0)
- moved C1 0.44 mm to (150.3, 131.3)
- moved SW1 0.20 mm to (123.5, 143.6)
Routing:
- net 5V: track 88.9 -> 179.0 mm, vias 2 -> 8
- net Net-(P2-Pad1): track 9.92 -> 81.9 mm, vias 0 -> 7
- net 3.3V: track 10.5 -> 73.3 mm, vias 0 -> 6
- net Net-(C3-Pad1): track 11.8 -> 44.4 mm, vias 1 -> 2
- net B1: track 4.14 -> 26.5 mm, vias 1 -> 2
- net GND: track 52.6 -> 70.0 mm, vias 13 -> 55
- net Net-(D3-Pad2): track 7.32 -> 11.5 mm, vias 0 -> 2
- net Net-(C17-Pad1): track 0.00 -> 2.00 mm
- net MOTOR_B_2: track 27.6 -> 28.9 mm
- net MOTOR_A_2: track 14.7 -> 15.6 mm
- net RST: track 23.9 -> 24.6 mm
- net MOTOR_A_1: track 15.0 -> 14.4 mm
- net Vusb: track 46.9 -> 47.1 mm, vias 3 -> 4
- net Net-(P4-Pad2): vias 2 -> 3
